Commit message: converted some URDFs to new SDF 1.5 compatible format
thanks to Michael Görner

File: uos_common_urdf/urdf/sick_lms200.urdf.xacro (robot description, xacro)
@@ -29,25 +29,31 @@
   <gazebo reference="laser">
     <material value="Gazebo/Blue" />
-    <sensor:ray name="laser">
-      <rayCount>181</rayCount>
-      <rangeCount>181</rangeCount>
-      <laserCount>1</laserCount>
-      <origin>0.0 0.0 0.0</origin>
-      <displayRays>false</displayRays>
-      <minAngle>-90</minAngle>
-      <maxAngle>90</maxAngle>
-      <minRange>0.08</minRange>
-      <maxRange>10.0</maxRange>
-      <resRange>0.01</resRange>
-      <updateRate>75.0</updateRate>
-      <controller:gazebo_ros_laser name="gazebo_ros_laser_controller" plugin="libgazebo_ros_laser.so">
+    <sensor type="ray" name="laser">
+      <always_on>true</always_on>
+      <visualize>false</visualize>
+      <topic>scan</topic>
+      <update_rate>75.0</update_rate>
+      <plugin name="gazebo_ros_laser_controller" filename="libgazebo_ros_laser.so">
+        <frameName>laser</frameName>
+        <topicName>scan</topicName>
         <gaussianNoise>0.005</gaussianNoise>
-        <alwaysOn>true</alwaysOn>
         <updateRate>75.0</updateRate>
-        <topicName>scan</topicName>
-        <frameName>laser</frameName>
-        <interface:laser name="gazebo_ros_laser_iface" />
-      </controller:gazebo_ros_laser>
-    </sensor:ray>
+      </plugin>
+      <ray>
+        <scan>
+          <horizontal>
+            <samples>181</samples>
+            <resolution>1</resolution>
+            <min_angle>-1.571</min_angle>
+            <max_angle>1.571</max_angle>
+          </horizontal>
+        </scan>
+        <range>
+          <min>0.08</min>
+          <max>10.0</max>
+          <resolution>0.01</resolution>
+        </range>
+      </ray>
+    </sensor>
   </gazebo>
 </robot>

Commit message: sick_lms200.urdf.xacro: link name is now set via macro

File: uos_common_urdf/urdf/sick_lms200.urdf.xacro (robot description, xacro)
@@ -4,56 +4,58 @@
   xmlns:sensor="http://playerstage.sourceforge.net/gazebo/xmlschema/#sensor"
   xmlns:xacro="http://ros.org/wiki/xacro">
-  <link name="laser">
-    <visual>
-      <geometry>
-        <mesh filename="package://uos_common_urdf/meshes/sick_lms-200.stl" />
-      </geometry>
-      <material name="blue" >
-        <color rgba="0 0 1 1" />
-      </material>
-    </visual>
-    <collision>
-      <geometry>
-        <mesh filename="package://uos_common_urdf/meshes/sick_lms-200.stl" />
-        <!-- <box size=".156 .155 .185" />-->
-      </geometry>
-    </collision>
-    <inertial>
-      <mass value="2.0" />
-      <origin xyz="-0.022849644 0.000005772 0.040232937" />
-      <inertia ixx="0.009318238" ixy="-0.000000024" ixz="-0.000148360"
-        iyy="0.009251799" iyz="0.000000400"
-        izz="0.007478235" />
-    </inertial>
-  </link>
-  <gazebo reference="laser">
-    <material value="Gazebo/Blue" />
-    <sensor type="ray" name="laser">
-      <always_on>true</always_on>
-      <visualize>false</visualize>
-      <topic>scan</topic>
-      <update_rate>75.0</update_rate>
-      <plugin name="gazebo_ros_laser_controller" filename="libgazebo_ros_laser.so">
-        <frameName>laser</frameName>
-        <topicName>scan</topicName>
-        <gaussianNoise>0.005</gaussianNoise>
-        <updateRate>75.0</updateRate>
-      </plugin>
-      <ray>
-        <scan>
-          <horizontal>
-            <samples>181</samples>
-            <resolution>1</resolution>
-            <min_angle>-1.571</min_angle>
-            <max_angle>1.571</max_angle>
-          </horizontal>
-        </scan>
-        <range>
-          <min>0.08</min>
-          <max>10.0</max>
-          <resolution>0.01</resolution>
-        </range>
-      </ray>
-    </sensor>
-  </gazebo>
+  <xacro:macro name="sick_lms200" params="laser_link">
+    <link name="${laser_link}">
+      <visual>
+        <geometry>
+          <mesh filename="package://uos_common_urdf/meshes/sick_lms-200.stl" />
+        </geometry>
+        <material name="blue" >
+          <color rgba="0 0 1 1" />
+        </material>
+      </visual>
+      <collision>
+        <geometry>
+          <mesh filename="package://uos_common_urdf/meshes/sick_lms-200.stl" />
+          <!-- <box size=".156 .155 .185" />-->
+        </geometry>
+      </collision>
+      <inertial>
+        <mass value="2.0" />
+        <origin xyz="-0.022849644 0.000005772 0.040232937" />
+        <inertia ixx="0.009318238" ixy="-0.000000024" ixz="-0.000148360"
+          iyy="0.009251799" iyz="0.000000400"
+          izz="0.007478235" />
+      </inertial>
+    </link>
+    <gazebo reference="${laser_link}">
+      <material value="Gazebo/Blue" />
+      <sensor type="ray" name="laser">
+        <always_on>true</always_on>
+        <visualize>false</visualize>
+        <topic>scan</topic>
+        <update_rate>75.0</update_rate>
+        <plugin name="gazebo_ros_laser_controller" filename="libgazebo_ros_laser.so">
+          <frameName>laser</frameName>
+          <topicName>scan</topicName>
+          <gaussianNoise>0.005</gaussianNoise>
+          <updateRate>75.0</updateRate>
+        </plugin>
+        <ray>
+          <scan>
+            <horizontal>
+              <samples>181</samples>
+              <resolution>1</resolution>
+              <min_angle>-1.571</min_angle>
+              <max_angle>1.571</max_angle>
+            </horizontal>
+          </scan>
+          <range>
+            <min>0.08</min>
+            <max>10.0</max>
+            <resolution>0.01</resolution>
+          </range>
+        </ray>
+      </sensor>
+    </gazebo>
+</xacro:macro>
 </robot>

Commit message: uos_common_urdf: add gazebo-topic parameter to sick_lms200 urdf file

File: uos_common_urdf/urdf/sick_lms200.urdf.xacro (robot description, xacro)
@@ -4,5 +4,5 @@
   xmlns:sensor="http://playerstage.sourceforge.net/gazebo/xmlschema/#sensor"
   xmlns:xacro="http://ros.org/wiki/xacro">
-  <xacro:macro name="sick_lms200" params="laser_link">
+  <xacro:macro name="sick_lms200" params="laser_link gazebo_topic">
     <link name="${laser_link}">
       <visual>
@@ -30,5 +30,5 @@
     <gazebo reference="${laser_link}">
       <material value="Gazebo/Blue" />
-      <sensor:ray name="laser">
+      <sensor:ray name="${laser_link}">
         <rayCount>181</rayCount>
         <rangeCount>181</rangeCount>
@@ -46,6 +46,6 @@
           <alwaysOn>true</alwaysOn>
           <updateRate>75.0</updateRate>
-          <topicName>scan</topicName>
-          <frameName>laser</frameName>
+          <topicName>${laser_link}</topicName>
+          <frameName>${gazebo_topic}</frameName>
           <interface:laser name="gazebo_ros_laser_iface" />
         </controller:gazebo_ros_laser>

Commit message: uos_common_urdf: add gazebo-topic parameter to sick_lms200 urdf file

File: uos_common_urdf/urdf/sick_lms200.urdf.xacro (robot description, xacro)
@@ -4,5 +4,5 @@
   xmlns:sensor="http://playerstage.sourceforge.net/gazebo/xmlschema/#sensor"
   xmlns:xacro="http://ros.org/wiki/xacro">
-  <xacro:macro name="sick_lms200" params="laser_link">
+  <xacro:macro name="sick_lms200" params="laser_link gazebo_topic">
     <link name="${laser_link}">
       <visual>
@@ -30,12 +30,11 @@
     <gazebo reference="${laser_link}">
       <material value="Gazebo/Blue" />
-      <sensor type="ray" name="laser">
+      <sensor type="ray" name="${laser_link}">
         <always_on>true</always_on>
         <visualize>false</visualize>
-        <topic>scan</topic>
         <update_rate>75.0</update_rate>
         <plugin name="gazebo_ros_laser_controller" filename="libgazebo_ros_laser.so">
-          <frameName>laser</frameName>
-          <topicName>scan</topicName>
+          <frameName>${laser_link}</frameName>
+          <topicName>${gazebo_topic}</topicName>
           <gaussianNoise>0.005</gaussianNoise>
           <updateRate>75.0</updateRate>
