Commit message: Rename package to uos_common_urdf

File: uos_common_urdf/urdf/kinect.urdf.xacro (robot description, xacro)
@@ -5,6 +5,6 @@
   xmlns:xacro="http://ros.org/wiki/xacro"
   name="${camera}">
-  <include filename="$(find kurt_description)/common.xacro" />
-  <include filename="$(find kurt_description)/parts/openni.gazebo.xacro" />
+  <include filename="$(find uos_common_urdf)/common.xacro" />
+  <include filename="$(find uos_common_urdf)/urdf/openni.gazebo.xacro" />
   <xacro:macro name="kinect" params="camera">
     <link name="${camera}_link">

File: uos_common_urdf/urdf/sick_lms100.urdf.xacro (robot description, xacro)
@@ -5,5 +5,5 @@
   xmlns:sensor="http://playerstage.sourceforge.net/gazebo/xmlschema/#sensor"
   >
-  <include filename="$(find kurt_description)/common.xacro" />
+  <include filename="$(find uos_common_urdf)/common.xacro" />
   <xacro:property name="laser_x" value="0.105" />
   <xacro:property name="laser_y" value="0.102" />
@@ -13,5 +13,5 @@
     <visual>
       <geometry>
-        <mesh filename="package://kurt_description/meshes/sick_lms-100.stl" />
+        <mesh filename="package://uos_common_urdf/meshes/sick_lms-100.stl" />
         <!-- <box size="${laser_x} ${laser_y} ${laser_z}" /> -->
       </geometry>
@@ -22,5 +22,5 @@
     <collision>
       <geometry>
-        <mesh filename="package://kurt_description/meshes/sick_lms-100.stl" />
+        <mesh filename="package://uos_common_urdf/meshes/sick_lms-100.stl" />
         <!-- <box size="${laser_x} ${laser_y} ${laser_z}" /> -->
       </geometry>

File: uos_common_urdf/urdf/sick_lms200.urdf.xacro (robot description, xacro)
@@ -7,5 +7,5 @@
     <visual>
       <geometry>
-        <mesh filename="package://kurt_description/meshes/sick_lms-200.stl" />
+        <mesh filename="package://uos_common_urdf/meshes/sick_lms-200.stl" />
       </geometry>
       <material name="blue" >
@@ -15,5 +15,5 @@
     <collision>
       <geometry>
-        <mesh filename="package://kurt_description/meshes/sick_lms-200.stl" />
+        <mesh filename="package://uos_common_urdf/meshes/sick_lms-200.stl" />
         <!-- <box size=".156 .155 .185" />-->
       </geometry>

File: uos_common_urdf/urdf/sick_s300.urdf.xacro (robot description, xacro)
@@ -2,5 +2,5 @@
 <robot
   xmlns:xacro="http://ros.org/wiki/xacro">
-  <include filename="$(find kurt_description)/common.xacro" />
+  <include filename="$(find uos_common_urdf)/common.xacro" />
   <xacro:property name="laser_x" value="0.156" />
   <xacro:property name="laser_y" value="0.155" />

Commit message: import pr2_description's kinect mesh
This makes uos_tools independent of pr2 modules

File: uos_common_urdf/urdf/kinect.urdf.xacro (robot description, xacro)
@@ -12,5 +12,5 @@
         <origin xyz="0 0 0" rpy="0 0 0" />
         <geometry>
-          <mesh filename="package://pr2_description/meshes/sensors/kinect_v0/kinect.dae" scale="0.001 0.001 0.001" />
+          <mesh filename="package://uos_common_urdf/meshes/kinect.dae" scale="0.001 0.001 0.001" />
         </geometry>
       </visual>
